Commit message: Change default joint positions

File: urdf/a1.urdf (robot description, URDF)
Before this commit: robot a1, 23 links, 22 joints
Joints:
- joint FL_thigh_joint: origin xyz=0 0.0838 0 rpy=0 0 0 -> xyz=0 0.0838 0 rpy=0 0.5 0
- joint FR_thigh_joint: origin xyz=0 -0.0838 0 rpy=0 0 0 -> xyz=0 -0.0838 0 rpy=0 0.5 0
- joint RL_thigh_joint: origin xyz=0 0.0838 0 rpy=0 0 0 -> xyz=0 0.0838 0 rpy=0 0.5 0
- joint RR_thigh_joint: origin xyz=0 -0.0838 0 rpy=0 0 0 -> xyz=0 -0.0838 0 rpy=0 0.5 0

File: xacro/leg.xacro (robot description, xacro)
@@ -65,5 +65,5 @@
         </link>
         <joint name="${name}_thigh_joint" type="revolute">
-            <origin rpy="0 0 0" xyz="0 ${thigh_offset*mirror} 0"/>
+            <origin rpy="0 0.5 0" xyz="0 ${thigh_offset*mirror} 0"/>
             <parent link="${name}_hip"/>
             <child link="${name}_thigh"/>
